File: PCB/Aeronet 5 to 4 serial.kicad_pcb (KiCad board)
At the start: 2 copper layers, 27.3 x 8.9 mm, 2 parts

Commit message: slight edit
Routing:
- net (no net): track 92.9 -> 101.3 mm
Changed lines of the file:
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@@
     (fp_line (start 5.08 -5.353039) (end -5.08 -5.353039) (layer "F.Fab") (width 0.1))
     (fp_line (start -2.175 -5.293039) (end 3.175 -5.293039) (layer "F.Fab") (width 0.1))
-    (pad "GND" smd rect (at -1 -4) (size 3.1 1.6) (layers "B.Cu" "B.Paste" "B.Mask"))
+    (pad "GND" smd rect (at -4.440096 -4.060224) (size 3.1 1.6) (layers "B.Cu" "B.Paste" "B.Mask"))
     (pad "RX" smd rect (at -4.445 0) (size 3.1 1.6) (layers "F.Cu" "F.Paste" "F.Mask"))
-    (pad "TS" smd rect (at -1 -1) (size 3.1 1.6) (layers "B.Cu" "B.Paste" "B.Mask"))
+    (pad "TS" smd rect (at -4.440096 -1.060224) (size 3.1 1.6) (layers "B.Cu" "B.Paste" "B.Mask"))
     (pad "TS" smd rect (at -4.445 -2.54) (size 3.1 1.6) (layers "F.Cu" "F.Paste" "F.Mask"))
-    (pad "TX" smd rect (at -0.90765 1.623987) (size 3.1 1.6) (layers "B.Cu" "B.Paste" "B.Mask"))
+    (pad "TX" smd rect (at -4.347746 1.563763) (size 3.1 1.6) (layers "B.Cu" "B.Paste" "B.Mask"))
     (model "${KICAD6_3DMODEL_DIR}/Package_DIP.3dshapes/DIP-10_W8.89mm_SMDSocket.wrl"
       (offset (xyz 0 0 0))
@@
   (gr_line (start 101.6 84.455) (end 101.6 91.44) (layer "Edge.Cuts") (width 0.2))
   (gr_line (start 88.9 84.455) (end 101.6 84.455) (layer "Edge.Cuts") (width 0.2))
-  (gr_text "Green\n" (at 84.502068 87.766868) (layer "B.SilkS")
+  (gr_text "Green\n" (at 82.316932 87.766868) (layer "B.SilkS")
     (effects (font (size 1.5 1.5) (thickness 0.3)) (justify mirror))
   )
-  (gr_text "Wh/Or" (at 84.502068 84.863331) (layer "B.SilkS")
+  (gr_text "Wh/Or" (at 82.316932 84.863331) (layer "B.SilkS")
     (effects (font (size 1.5 1.5) (thickness 0.3)) (justify mirror))
   )
@@
     (effects (font (size 1.5 1.5) (thickness 0.3)) (justify mirror))
   )
-  (gr_text "Blue" (at 85.370136 90.341139) (layer "B.SilkS")
+  (gr_text "Blue" (at 83.185 90.341139) (layer "B.SilkS")
     (effects (font (size 1.5 1.5) (thickness 0.3)) (justify mirror))
   )
@@
   )
   (segment (start 90.805 86.995) (end 91.128979 87.318979) (width 0.25) (layer "F.Cu") (net 0))
-  (segment (start 76.2 87.63) (end 76.2 86.36) (width 0.25) (layer "F.Cu") (net 0))
+  (segment (start 79.01 87.9) (end 77.47 86.36) (width 0.25) (layer "F.Cu") (net 0))
+  (segment (start 77.47 86.36) (end 76.2 86.36) (width 0.25) (layer "F.Cu") (net 0))
   (segment (start 91.128979 87.318979) (end 99.502695 87.318979) (width 0.25) (layer "F.Cu") (net 0))
   (segment (start 89.535 88.9) (end 76.2 88.9) (width 0.25) (layer "F.Cu") (net 0))
@@
   (segment (start 90.805 90.17) (end 98.940287 90.17) (width 0.25) (layer "F.Cu") (net 0))
   (segment (start 98.940287 90.17) (end 99.543485 89.566802) (width 0.25) (layer "F.Cu") (net 0))
-  (via (at 76.2 87.63) (size 0.8) (drill 0.4) (layers "F.Cu" "B.Cu") (net 0))
+  (via (at 79.01 87.9) (size 0.8) (drill 0.4) (layers "F.Cu" "B.Cu") (net 0))
   (via (at 90.805 90.17) (size 0.8) (drill 0.4) (layers "F.Cu" "B.Cu") (net 0))
   (via (at 89.535 88.9) (size 0.8) (drill 0.4) (layers "F.Cu" "B.Cu") (net 0))
-  (segment (start 80.991158 86.246158) (end 79.645 84.9) (width 0.25) (layer "B.Cu") (net 0))
-  (segment (start 76.2 87.63) (end 76.47 87.9) (width 0.25) (layer "B.Cu") (net 0))
-  (segment (start 99.483874 86.253446) (end 99.476586 86.246158) (width 0.25) (layer "B.Cu") (net 0))
+  (segment (start 79.584776 84.839776) (end 80.991158 86.246158) (width 0.25) (layer "B.Cu") (net 0))
   (segment (start 99.521517 88.474372) (end 99.521517 88.944908) (width 0.25) (layer "B.Cu") (net 0))
-  (segment (start 79.73735 90.523987) (end 88.546013 90.523987) (width 0.25) (layer "B.Cu") (net 0))
-  (segment (start 76.47 87.9) (end 79.645 87.9) (width 0.25) (layer "B.Cu") (net 0))
-  (segment (start 99.476586 86.246158) (end 80.991158 86.246158) (width 0.25) (layer "B.Cu") (net 0))
-  (segment (start 88.9 90.17) (end 90.805 90.17) (width 0.25) (layer "B.Cu") (net 0))
+  (segment (start 80.991158 86.246158) (end 99.476586 86.246158) (width 0.25) (layer "B.Cu") (net 0))
+  (segment (start 76.297254 90.463763) (end 76.357478 90.523987) (width 0.25) (layer "B.Cu") (net 0))
+  (segment (start 76.265128 87.9) (end 76.204904 87.839776) (width 0.25) (layer "B.Cu") (net 0))
+  (segment (start 76.204904 84.839776) (end 79.584776 84.839776) (width 0.25) (layer "B.Cu") (net 0))
   (segment (start 88.546013 90.523987) (end 88.9 90.17) (width 0.25) (layer "B.Cu") (net 0))
   (segment (start 99.521517 88.944908) (end 99.476609 88.9) (width 0.25) (layer "B.Cu") (net 0))
+  (segment (start 79.01 87.9) (end 76.265128 87.9) (width 0.25) (layer "B.Cu") (net 0))
+  (segment (start 88.9 90.17) (end 90.805 90.17) (width 0.25) (layer "B.Cu") (net 0))
   (segment (start 99.476609 88.9) (end 89.535 88.9) (width 0.25) (layer "B.Cu") (net 0))
+  (segment (start 76.357478 90.523987) (end 88.546013 90.523987) (width 0.25) (layer "B.Cu") (net 0))
+  (segment (start 99.476586 86.246158) (end 99.483874 86.253446) (width 0.25) (layer "B.Cu") (net 0))
   (group "" (id 4736c914-4475-4c5e-8038-2dadbdab8425)
     (members
